File: experience/keebored/keebored/RPI-RP2040-MINIMAL_R3-S1.kicad_pcb (KiCad board)
At the start: 2 copper layers, 55 x 95 mm, 66 parts, among them J1 USB_C_Receptacle_USB2.0_16P, J2 TSW-102-07-G-S, J3 Conn_01x04_Socket, J4 Conn_01x03_Pin, SW1 SW_Push, SW2 RotaryEncoder_Switch_MP, U1 NCP1117ST33T3G, U2 W25Q128JVSIQ, U3 RP2040, U4 TPD2E2U06DRL, X1 12MHz

Commit message: c
Parts:
- moved J2 33.8 mm to (43.6, 46.7), turned to 0 degrees
- moved R1 29.3 mm to (41.2, 48.5)
- moved R2 29.3 mm to (39.7, 48.5)
- moved C17 25.9 mm to (43.6, 34.1)
- moved C5 25.9 mm to (48.9, 36.4)
- moved U2 25.9 mm to (46.8, 40.0)
- moved X1 21.2 mm to (16.5, 43.9), turned to -90 degrees
- moved C2 17.9 mm to (19.3, 42.6), turned to 90 degrees
- moved C3 17.0 mm to (19.3, 45.2), turned to -90 degrees
- moved C27 14.6 mm to (37.2, 6.80)
- moved J3 14.1 mm to (35.0, 4.50)
- moved J4 13.8 mm to (47.2, 71.4), turned to -90 degrees
- moved R5 13.6 mm to (22.3, 43.2), turned to 0 degrees
- moved R13 13.5 mm to (46.8, 82.6), turned to 0 degrees
- moved C14 13.1 mm to (22.3, 44.3), turned to 180 degrees
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Routing:
- net Net-(LED3-CKO): track 0.00 -> 45.7 mm
- net Net-(LED3-SDO): track 0.00 -> 40.8 mm
- net /USB_D+: track 10.8 -> 50.3 mm, vias 0 -> 2
- net Net-(LED2-SDO): track 0.00 -> 39.0 mm
- net /GPIO29_ADC3: track 0.00 -> 38.4 mm, vias 0 -> 1
- net /GPIO28_ADC2: track 0.01 -> 36.9 mm, vias 0 -> 1
- net /USB_D-: track 17.3 -> 53.0 mm
- net Net-(LED2-CKO): track 0.00 -> 33.3 mm
- net /GPIO0: track 1.99 -> 30.9 mm, vias 0 -> 2
- net /GPIO1: track 1.90 -> 26.5 mm, vias 0 -> 2
- net Net-(LED1-CKO): track 0.00 -> 24.1 mm
- net /GPIO9: track 63.0 -> 39.2 mm
- net Net-(LED1-SDO): track 0.00 -> 23.2 mm
- net +3V3: track 29.9 -> 52.6 mm, vias 2 -> 19
- net /GPIO8: track 63.5 -> 40.9 mm
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Other:
- board text removed: "Minimal Design Example R3"
- board text removed: "Raspberry Pi RP2040"
